File: MAX31790-Breakout-Board.kicad_sch (KiCad schematic)
At the start: 26 parts, among them J1 Conn_01x07, J2 Conn_01x05, J3 Screw_Terminal_01x02, M1 Fan_4pin, M2 Fan_4pin, M3 Fan_4pin, M4 Fan_4pin, M5 Fan_4pin, M6 Fan_4pin, U1 MAX31790ATI_T

Commit message: Added +12V line for fan power
Parts:
- removed J3: Screw_Terminal_01x02, TerminalBlock_Phoenix:TerminalBlock_Phoenix_MKDS-1,5-2-5.08_1x02_P5.08mm_Horizontal, symbol Connector:Screw_Terminal_01x02
- added C2: 1uF, Capacitor_SMD:C_0603_1608Metric, symbol Device:C
- added J3: Screw_Terminal_01x03, TerminalBlock_Phoenix:TerminalBlock_Phoenix_MPT-0,5-3-2.54_1x03_P2.54mm_Horizontal, symbol Connector:Screw_Terminal_01x03
Connections:
- net +3V3: now also J3.2 (Pin_2); no longer M1.2 (+), M2.2 (+), M3.2 (+), M4.2 (+), M5.2 (+), M6.2 (+)
- net GND: now also U1.29 (EXPPAD), C2.2, J3.3 (Pin_3)
- new net +12V: C2.1, J3.1 (Pin_1), M1.2 (+), M2.2 (+), M3.2 (+), M4.2 (+), M5.2 (+), M6.2 (+)
Other:
- moved on the sheet: C1, U1

Commit message: Added page settings
Other:
- company: (none) -> Rolando Rosales
- title: (none) -> MAX31790 Breakout Board
Changed lines of the file:
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@@
 	(generator_version "8.0")
 	(paper "A4")
+	(title_block
+		(title "MAX31790 Breakout Board")
+		(date "2024-06-07")
+		(rev "0.1")
+		(company "Rolando Rosales")
+		(comment 1 "https://github.com/rolo-g/MAX31790-Breakout-Board")
+	)
 	(junction
 		(at 182.88 59.69)
